File: hardware/project-embeddedSystemDesign2/project-embeddedSystemDesign2.kicad_pcb (KiCad board)
At the start: 2 copper layers, 58.4 x 64.8 mm, 41 parts, among them J1 Conn_02x04_Odd_Even, J10 Conn_02x02_Odd_Even, J11 Conn_01x03, J12 Conn_01x02, J2 Conn_02x09_Odd_Even, J3 Conn_01x04, J4 Conn_02x02_Odd_Even, J5 Conn_02x02_Odd_Even, J6 Conn_01x03, J7 Conn_01x02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

Commit message: Update PCB
Other:
- board text added: "EFM32HG322: 1.98 - 3.8V ADXL362: 1.6 - 3.5V DS18B20: 3 - 5.5V"
- board text added: "MIN 3.0V"
- board text added: "X"
- board text added: "Y"
- board text added: "Z"
Changed lines of the file:
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@@
   (general
     (thickness 1.6)
-    (drawings 52)
+    (drawings 71)
     (tracks 433)
     (zones 0)
@@
     (visible_elements FFFDFF7F)
     (pcbplotparams
-      (layerselection 0x00020_7ffffffe)
+      (layerselection 0x00040_fffffffe)
       (usegerberextensions false)
       (usegerberattributes false)
@@
       (psa4output false)
       (plotreference true)
-      (plotvalue true)
+      (plotvalue false)
       (plotinvisibletext false)
       (padsonsilk false)
-      (subtractmaskfromsilk false)
+      (subtractmaskfromsilk true)
       (outputformat 4)
       (mirror true)
       (drillshape 0)
       (scaleselection 1)
-      (outputdirectory ""))
+      (outputdirectory "pdf/"))
   )
   (net 0 "")
@@
       (net 1 GND) (solder_mask_margin 0.1016))
   )
+  (gr_text "EFM32HG322: 1.98 - 3.8V\nADXL362: 1.6 - 3.5V\nDS18B20: 3 - 5.5V" (at 127 92.71) (layer B.Paste)
+    (effects (font (size 1 1) (thickness 0.15)) (justify mirror))
+  )
+  (gr_text "MIN 3.0V" (at 112.776 47.752 270) (layer F.SilkS)
+    (effects (font (size 1 1) (thickness 0.15)) (justify right))
+  )
+  (dimension 3.048 (width 0.15) (layer Dwgs.User)
+    (gr_text "3,048 mm" (at 159.034 100.33 270) (layer Dwgs.User)
+      (effects (font (size 1 1) (thickness 0.15)))
+    )
+    (feature1 (pts (xy 152.4 101.854) (xy 158.320421 101.854)))
+    (feature2 (pts (xy 152.4 98.806) (xy 158.320421 98.806)))
+    (crossbar (pts (xy 157.734 98.806) (xy 157.734 101.854)))
+    (arrow1a (pts (xy 157.734 101.854) (xy 157.147579 100.727496)))
+    (arrow1b (pts (xy 157.734 101.854) (xy 158.320421 100.727496)))
+    (arrow2a (pts (xy 157.734 98.806) (xy 157.147579 99.932504)))
+    (arrow2b (pts (xy 157.734 98.806) (xy 158.320421 99.932504)))
+  )
+  (dimension 57.15 (width 0.15) (layer Dwgs.User)
+    (gr_text "57,150 mm" (at 92.68 71.755 270) (layer Dwgs.User)
+      (effects (font (size 1 1) (thickness 0.15)))
+    )
+    (feature1 (pts (xy 101.6 100.33) (xy 93.393579 100.33)))
+    (feature2 (pts (xy 101.6 43.18) (xy 93.393579 43.18)))
+    (crossbar (pts (xy 93.98 43.18) (xy 93.98 100.33)))
+    (arrow1a (pts (xy 93.98 100.33) (xy 93.393579 99.203496)))
+    (arrow1b (pts (xy 93.98 100.33) (xy 94.566421 99.203496)))
+    (arrow2a (pts (xy 93.98 43.18) (xy 93.393579 44.306504)))
+    (arrow2b (pts (xy 93.98 43.18) (xy 94.566421 44.306504)))
+  )
+  (dimension 64.77 (width 0.15) (layer Dwgs.User)
+    (gr_text "64,770 mm" (at 162.59 71.755 270) (layer Dwgs.User)
+      (effects (font (size 1 1) (thickness 0.15)))
+    )
+    (feature1 (pts (xy 156.21 104.14) (xy 161.876421 104.14)))
+    (feature2 (pts (xy 156.21 39.37) (xy 161.876421 39.37)))
+    (crossbar (pts (xy 161.29 39.37) (xy 161.29 104.14)))
+    (arrow1a (pts (xy 161.29 104.14) (xy 160.703579 103.013496)))
+    (arrow1b (pts (xy 161.29 104.14) (xy 161.876421 103.013496)))
+    (arrow2a (pts (xy 161.29 39.37) (xy 160.703579 40.496504)))
+    (arrow2b (pts (xy 161.29 39.37) (xy 161.876421 40.496504)))
+  )
+  (dimension 50.8 (width 0.15) (layer Dwgs.User)
+    (gr_text "50,800 mm" (at 127 108.996) (layer Dwgs.User)
+      (effects (font (size 1 1) (thickness 0.15)))
+    )
+    (feature1 (pts (xy 152.4 100.33) (xy 152.4 108.282421)))
+    (feature2 (pts (xy 101.6 100.33) (xy 101.6 108.282421)))
+    (crossbar (pts (xy 101.6 107.696) (xy 152.4 107.696)))
+    (arrow1a (pts (xy 152.4 107.696) (xy 151.273496 108.282421)))
+    (arrow1b (pts (xy 152.4 107.696) (xy 151.273496 107.109579)))
+    (arrow2a (pts (xy 101.6 107.696) (xy 102.726504 108.282421)))
+    (arrow2b (pts (xy 101.6 107.696) (xy 102.726504 107.109579)))
+  )
+  (gr_line (start 98.552 52.07) (end 103.886 52.07) (layer F.SilkS) (width 0.12))
+  (gr_line (start 98.552 46.228) (end 98.552 52.07) (layer F.SilkS) (width 0.12))
+  (gr_line (start 103.886 46.228) (end 98.552 46.228) (layer F.SilkS) (width 0.12))
+  (gr_line (start 103.886 52.07) (end 103.886 46.228) (layer F.SilkS) (width 0.12))
+  (gr_line (start 101.346 50.546) (end 99.822 50.546) (layer F.SilkS) (width 0.12))
+  (gr_line (start 99.822 50.546) (end 100.33 50.038) (layer F.SilkS) (width 0.12))
+  (gr_line (start 99.822 50.546) (end 100.33 51.054) (layer F.SilkS) (width 0.12))
+  (gr_line (start 102.362 48.006) (end 101.854 48.514) (layer F.SilkS) (width 0.12))
+  (gr_line (start 102.362 48.006) (end 102.87 48.514) (layer F.SilkS) (width 0.12))
+  (gr_line (start 102.362 49.53) (end 102.362 48.006) (layer F.SilkS) (width 0.12))
+  (gr_circle (center 102.362 50.546) (end 103.378 50.546) (layer F.SilkS) (width 0.12))
+  (gr_text Z (at 102.362 50.546) (layer F.SilkS)
+    (effects (font (size 1 1) (thickness 0.15)))
+  )
+  (gr_text Y (at 99.314 50.546) (layer F.SilkS)
+    (effects (font (size 1 1) (thickness 0.15)))
+  )
+  (gr_text X (at 102.362 47.244) (layer F.SilkS)
+    (effects (font (size 1 1) (thickness 0.15)))
+  )
   (gr_text "MAX 3.5V" (at 105.41 48.006 270) (layer F.SilkS)
     (effects (font (size 1 1) (thickness 0.15)) (justify right))
@@
     (effects (font (size 1 1) (thickness 0.2)))
   )
-  (dimension 64.77 (width 0.12) (layer Dwgs.User)
-    (gr_text "64,770 mm" (at 91.44 71.755 90) (layer Dwgs.User)
-      (effects (font (size 1 1) (thickness 0.15)))
-    )
-    (feature1 (pts (xy 97.79 39.37) (xy 92.123579 39.37)))
-    (feature2 (pts (xy 97.79 104.14) (xy 92.123579 104.14)))
-    (crossbar (pts (xy 92.71 104.14) (xy 92.71 39.37)))
-    (arrow1a (pts (xy 92.71 39.37) (xy 93.296421 40.496504)))
-    (arrow1b (pts (xy 92.71 39.37) (xy 92.123579 40.496504)))
-    (arrow2a (pts (xy 92.71 104.14) (xy 93.296421 103.013496)))
-    (arrow2b (pts (xy 92.71 104.14) (xy 92.123579 103.013496)))
-  )
   (dimension 58.42 (width 0.12) (layer Dwgs.User)
